File: kicad/Palette58_left/Palette58_left.kicad_sch (KiCad schematic)
At the start: 62 parts, among them SW1 SW_DPDT_x2, SW2 SW_Push

Commit message: Simplify left half
Parts:
- removed C1, C10, C11, C12, C13, C14, C15, C16, C17, C18, C19, C2, C20, C21, C22, C23, C24, C25, C26, C27, C28, C3, C4, C5, C6, C7, C8, C9: 100nF, symbol Device:C
- removed D30: 1N5819, symbol Device:D
- removed LED1, LED10, LED11, LED12, LED13, LED14, LED15, LED16, LED17, LED18, LED19, LED2, LED20, LED21, LED22, LED23, LED24, LED25, LED26, LED27, LED28, LED29, LED3, LED4, LED5, LED6, LED7, LED8, LED9: XINGLIGHTXL-1615RGBC-WS2812B, LED_SMD:XINGLIGHT XL-1615RGBC-WS2812B, symbol LED:WS2812B
- removed R1: 330Ω, Resistor_SMD:R_0402_1005Metric, symbol Device:R
- removed R2: 10kΩ, symbol Device:R
Connections:
- no-connect marks 2 -> 1
Other:
- moved on the sheet: SW1A, SW2
