File: kicad/Palette58_right/Palette58_right.kicad_sch (KiCad schematic)
At the start: 62 parts, among them SW1 SW_DPDT_x2, SW2 SW_Push

Commit message: Update right half
Parts:
- removed C1, C11, C13, C15, C17, C19, C21, C23, C25, C27, C29, C3, C31, C33, C35, C37, C39, C41, C43, C45, C47, C49, C5, C51, C53, C55, C7, C9: 100nF, symbol Device:C
- removed D30: 1N5819, symbol Device:D
- removed LED1, LED10, LED11, LED12, LED13, LED14, LED15, LED16, LED17, LED18, LED19, LED2, LED20, LED21, LED22, LED23, LED24, LED25, LED26, LED27, LED28, LED29, LED3, LED4, LED5, LED6, LED7, LED8, LED9: XINGLIGHTXL-1615RGBC-WS2812B, LED_SMD:XINGLIGHT XL-1615RGBC-WS2812B, symbol LED:WS2812B
- removed R1: 330Ω, Resistor_SMD:R_0402_1005Metric, symbol Device:R
- removed R2: 10kΩ, symbol Device:R
Connections:
- no-connect marks 2 -> 1
Other:
- moved on the sheet: SW1A, SW2
